File: Test_1_Hellen1.kicad_sch (KiCad schematic)
At the start: 2 parts, among them J1 Conn_01x07, M1 Module-can-0.1

Commit message: Aggiunto gerber\
Parts:
- M1: footprint hellen-one-can-0.1:can -> 0.1:can
Changed lines of the file:
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@@
 			)
 		)
-		(property "Footprint" "hellen-one-can-0.1:can"
+		(property "Footprint" "0.1:can"
 			(at 121.92 100.33 0)
 			(effects
